Commit message: Moved cassie class into folder. Added functions for IMU kinematics export

File: urdf/cassie_with_sensors.urdf (robot description, URDF)
Before this commit: robot cassie, 19 links, 18 joints
Joints:
- joint knee_to_shin_left: limit lower=0 upper=0 effort=0 velocity=0 -> lower=-100 upper=100 effort=0 velocity=100
- joint knee_to_shin_right: limit lower=0 upper=0 effort=0 velocity=0 -> lower=-100 upper=100 effort=0 velocity=100

File: urdf/cassie_with_sensors.xacro (robot description, xacro)
@@ -312,5 +312,5 @@
       <parent link="${side}_knee" />
       <child link="${side}_shin" />
-      <limit lower="0" upper="0" effort="0" velocity="0" />
+      <limit lower="-100" upper="100" effort="0" velocity="100" />
     </joint>
   </xacro:macro>

Commit message: rotated the IMU frame because Agility prerotates the data

File: urdf/cassie_with_sensors.urdf (robot description, URDF)
Before this commit: robot cassie, 19 links, 18 joints
Joints:
- joint fixed_pelvis_to_vectorNav: origin xyz=0.03155 0 -0.07996 rpy=3.14159265359 0 0 -> xyz=0.03155 0 -0.07996 rpy=0 0 0

File: urdf/cassie_with_sensors.xacro (robot description, xacro)
@@ -253,5 +253,5 @@
   <xacro:macro name="fixed_pelvis_to_vectorNav">
     <joint name="fixed_pelvis_to_vectorNav" type="fixed">
-      <origin xyz="0.03155 0 -0.07996" rpy="${pi} 0 0"/>
+      <origin xyz="0.03155 0 -0.07996" rpy="0 0 0"/>
       <parent link="pelvis" />
       <child link="vectorNav" />
